File: de0-nano_RMII.sch (EAGLE design)
At the start: 34 parts, among them U1 DP83848, X1 1-227161-2

Commit message: almost done
Parts:
- removed X4: (no value), con-lstb:MA04-1
- added J1: (no value), con-jack:JACK-PLUG1
- added J2: (no value), seeed_connector:JACK-3P-2.5MM-2.5MM
- added J3: (no value), seeed_connector:HEADER-4P-60/35MIL
Connections:
- new net VCC_SYS: J3.P$1, J3.P$2
- net GND: now also J1.1, J1.2, J3.P$3, J3.P$4
- net OSCIN: now also X2.17
- net RXD_0: now also X2.33
- net RXD_1: now also X2.34
- net TXD_0: now also X2.39
- net TXD_1: now also X2.40
- net TX_EN: now also X2.37
Other:
- moved on the sheet: C13, R14
Changed lines of the file:
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@@
 <?xml version="1.0" encoding="utf-8"?>
 <!DOCTYPE eagle SYSTEM "eagle.dtd">
-<eagle version="8.0.1">
+<eagle version="8.0.2">
 <drawing>
 <settings>
@@
 <setting verticaltext="up"/>
 </settings>
-<grid distance="0.05" unitdist="inch" unit="inch" style="lines" multiple="1" display="yes" altdistance="0.01" altunitdist="inch" altunit="inch"/>
+<grid distance="0.05" unitdist="inch" unit="inch" style="lines" multiple="1" display="no" altdistance="0.01" altunitdist="inch" altunit="inch"/>
 <layers>
 <layer number="1" name="Top" color="4" fill="1" visible="no" active="no"/>
@@
 <part name="X2" library="con-lstb" deviceset="MA20-2" device=""/>
 <part name="X3" library="con-lstb" deviceset="MA20-2" device=""/>
-<part name="X4" library="con-lstb" deviceset="MA04-1" device=""/>
 <part name="X7" library="seeed_connector" deviceset="RJ45-HR911105A" device="-HR911105A"/>
 <part name="U1" library="national-semiconductor" deviceset="DP83848" device=""/>
@@
 <part name="C13" library="resistor" deviceset="C-EU" device="C0805" value="10uF"/>
 <part name="GND16" library="supply1" deviceset="GND" device=""/>
+<part name="J1" library="con-jack" deviceset="JACK-PLUG" device="1"/>
+<part name="J2" library="seeed_connector" deviceset="JACK-3P-2.5MM" device="-2.5MM"/>
+<part name="J3" library="seeed_connector" deviceset="HEADER-4P" device="-60/35MIL"/>
+<part name="GND17" library="supply1" deviceset="GND" device=""/>
+<part name="GND18" library="supply1" deviceset="GND" device=""/>
 </parts>
 <sheets>
@@
 <instance part="X2" gate="G$1" x="45.72" y="125.73" rot="R180"/>
 <instance part="X3" gate="G$1" x="45.72" y="52.07" rot="R180"/>
-<instance part="X4" gate="1" x="257.81" y="85.09" rot="R180"/>
 <instance part="X7" gate="G$1" x="304.8" y="148.59"/>
 <instance part="U1" gate="G$1" x="172.72" y="130.81" smashed="yes">
@@
 <instance part="GND14" gate="1" x="55.88" y="97.79"/>
 <instance part="GND15" gate="1" x="55.88" y="24.13"/>
-<instance part="R14" gate="G$1" x="30.48" y="115.57" smashed="yes">
-<attribute name="NAME" x="27.94" y="117.0686" size="1.778" layer="95"/>
-<attribute name="VALUE" x="27.94" y="112.268" size="1.778" layer="96"/>
-</instance>
-<instance part="C13" gate="G$1" x="22.86" y="110.49" smashed="yes">
-<attribute name="NAME" x="16.764" y="110.871" size="1.778" layer="95"/>
-<attribute name="VALUE" x="16.764" y="105.791" size="1.778" layer="96"/>
-</instance>
-<instance part="GND16" gate="1" x="22.86" y="100.33"/>
+<instance part="R14" gate="G$1" x="22.86" y="115.57" smashed="yes">
+<attribute name="NAME" x="20.32" y="117.0686" size="1.778" layer="95"/>
+<attribute name="VALUE" x="20.32" y="112.268" size="1.778" layer="96"/>
+</instance>
+<instance part="C13" gate="G$1" x="15.24" y="110.49" smashed="yes">
+<attribute name="NAME" x="9.144" y="110.871" size="1.778" layer="95"/>
+<attribute name="VALUE" x="9.144" y="105.791" size="1.778" layer="96"/>
+</instance>
+<instance part="GND16" gate="1" x="15.24" y="100.33"/>
+<instance part="J1" gate="G$1" x="92.71" y="180.34"/>
+<instance part="J2" gate="G$1" x="123.19" y="186.69"/>
+<instance part="J3" gate="G$1" x="45.72" y="227.33" rot="R180"/>
+<instance part="GND17" gate="1" x="67.31" y="231.14" rot="R90"/>
+<instance part="GND18" gate="1" x="100.33" y="172.72"/>
 </instances>
 <busses>
@@
 <pinref part="GND16" gate="1" pin="GND"/>
 <pinref part="C13" gate="G$1" pin="2"/>
-<wire x1="22.86" y1="102.87" x2="22.86" y2="105.41" width="0.1524" layer="91"/>
+<wire x1="15.24" y1="102.87" x2="15.24" y2="105.41" width="0.1524" layer="91"/>
+</segment>
+<segment>
+<pinref part="J3" gate="G$1" pin="P$4"/>
+<pinref part="GND17" gate="1" pin="GND"/>
+<wire x1="53.34" y1="231.14" x2="55.88" y2="231.14" width="0.1524" layer="91"/>
+<pinref part="J3" gate="G$1" pin="P$3"/>
+<wire x1="55.88" y1="231.14" x2="64.77" y2="231.14" width="0.1524" layer="91"/>
+<wire x1="53.34" y1="228.6" x2="55.88" y2="228.6" width="0.1524" layer="91"/>
+<wire x1="55.88" y1="228.6" x2="55.88" y2="231.14" width="0.1524" layer="91"/>
+<junction x="55.88" y="231.14"/>
+</segment>
+<segment>
+<pinref part="J1" gate="G$1" pin="2"/>
+<pinref part="GND18" gate="1" pin="GND"/>
+<wire x1="97.79" y1="180.34" x2="100.33" y2="180.34" width="0.1524" layer="91"/>
+<wire x1="100.33" y1="180.34" x2="100.33" y2="177.8" width="0.1524" layer="91"/>
+<pinref part="J1" gate="G$1" pin="1"/>
+<wire x1="100.33" y1="177.8" x2="100.33" y2="175.26" width="0.1524" layer="91"/>
+<wire x1="97.79" y1="177.8" x2="100.33" y2="177.8" width="0.1524" layer="91"/>
+<junction x="100.33" y="177.8"/>
 </segment>
 </net>
@@
 <wire x1="137.16" y1="120.65" x2="121.92" y2="120.65" width="0.1524" layer="91"/>
 <label x="124.46" y="120.65" size="1.778" layer="95"/>
+</segment>
+<segment>
+<pinref part="X2" gate="G$1" pin="17"/>
+<wire x1="38.1" y1="130.81" x2="19.05" y2="130.81" width="0.1524" layer="91"/>
+<label x="24.13" y="130.81" size="1.778" layer="95"/>
 </segment>
 </net>
@@
 <segment>
 <pinref part="C13" gate="G$1" pin="1"/>
-<wire x1="22.86" y1="113.03" x2="22.86" y2="115.57" width="0.1524" layer="91"/>
+<wire x1="15.24" y1="113.03" x2="15.24" y2="115.57" width="0.1524" layer="91"/>
 <pinref part="R14" gate="G$1" pin="1"/>
-<wire x1="22.86" y1="115.57" x2="25.4" y2="115.57" width="0.1524" layer="91"/>
-<wire x1="13.97" y1="115.57" x2="22.86" y2="115.57" width="0.1524" layer="91"/>
-<junction x="22.86" y="115.57"/>
+<wire x1="15.24" y1="115.57" x2="17.78" y2="115.57" width="0.1524" layer="91"/>
+<wire x1="6.35" y1="115.57" x2="15.24" y2="115.57" width="0.1524" layer="91"/>
+<junction x="15.24" y="115.57"/>
 </segment>
 </net>
@@
 <label x="208.28" y="118.11" size="1.778" layer="95"/>
 </segment>
+<segment>
+<pinref part="X2" gate="G$1" pin="37"/>
+<wire x1="38.1" y1="105.41" x2="25.4" y2="105.41" width="0.1524" layer="91"/>
+<label x="27.94" y="105.41" size="1.778" layer="95"/>
+</segment>
 </net>
 <net name="TXD_0" class="0">
@@
 <label x="208.28" y="120.65" size="1.778" layer="95"/>
 </segment>
+<segment>
+<pinref part="X2" gate="G$1" pin="39"/>
+<wire x1="38.1" y1="102.87" x2="25.4" y2="102.87" width="0.1524" layer="91"/>
+<label x="27.94" y="102.87" size="1.778" layer="95"/>
+</segment>
 </net>
 <net name="TXD_1" class="0">
@@
 <label x="208.28" y="123.19" size="1.778" layer="95"/>
 </segment>
+<segment>
+<pinref part="X2" gate="G$1" pin="40"/>
+<wire x1="53.34" y1="102.87" x2="69.85" y2="102.87" width="0.1524" layer="91"/>
+<label x="58.42" y="102.87" size="1.778" layer="95"/>
+</segment>
 </net>
 <net name="RXD_0" class="0">
@@
 <label x="172.72" y="95.25" size="1.778" layer="95" rot="R90"/>
 </segment>
+<segment>
+<pinref part="X2" gate="G$1" pin="33"/>
+<wire x1="38.1" y1="110.49" x2="25.4" y2="110.49" width="0.1524" layer="91"/>
+<label x="27.94" y="110.49" size="1.778" layer="95"/>
+</segment>
 </net>
 <net name="RXD_1" class="0">
@@
 <wire x1="175.26" y1="105.41" x2="175.26" y2="92.71" width="0.1524" layer="91"/>
 <label x="175.26" y="95.25" size="1.778" layer="95" rot="R90"/>
+</segment>
+<segment>
+<pinref part="X2" gate="G$1" pin="34"/>
+<wire x1="53.34" y1="110.49" x2="69.85" y2="110.49" width="0.1524" layer="91"/>
+<label x="58.42" y="110.49" size="1.778" layer="95"/>
 </segment>
 </net>
@@
 <pinref part="R14" gate="G$1" pin="2"/>
 <pinref part="X2" gate="G$1" pin="29"/>
-<wire x1="35.56" y1="115.57" x2="38.1" y2="115.57" width="0.1524" layer="91"/>
-</segment>
-</net>
+<wire x1="27.94" y1="115.57" x2="38.1" y2="115.57" width="0.1524" layer="91"/>
+</segment>
+</net>
+<net name="VCC_SYS" class="0">
+<segment>
+<pinref part="J3" gate="G$1" pin="P$2"/>
+<wire x1="53.34" y1="226.06" x2="55.88" y2="226.06" width="0.1524" layer="91"/>
+<wire x1="55.88" y1="226.06" x2="55.88" y2="223.52" width="0.1524" layer="91"/>
+<pinref part="J3" gate="G$1" pin="P$1"/>
+<wire x1="55.88" y1="223.52" x2="53.34" y2="223.52" width="0.1524" layer="91"/>
+<wire x1="55.88" y1="223.52" x2="71.12" y2="223.52" width="0.1524" layer="91"/>
+<junction x="55.88" y="223.52"/>
+<label x="58.42" y="223.52" size="1.778" layer="95"/>
+</segment>
+</net>

Commit message: RX_DV and CRS_DV added
Connections:
- removed net N$1: R3.1, U1.RX_DV
- removed net N$2: R4.1, U1.CRS
- new net CRS_DV: R4.1, U1.CRS, X2.34
- new net RX_DV: R3.1, U1.RX_DV, X2.33
- net RXD_0: now also X2.35; no longer X2.33
- net RXD_1: now also X2.36; no longer X2.34
Other:
- moved on the sheet: R3, R4
Changed lines of the file:
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@@
 <instance part="GND4" gate="1" x="260.35" y="118.11"/>
 <instance part="GND5" gate="1" x="260.35" y="167.64" rot="R180"/>
-<instance part="R3" gate="G$1" x="152.4" y="92.71" smashed="yes" rot="R180">
-<attribute name="NAME" x="147.32" y="94.2086" size="1.778" layer="95"/>
-<attribute name="VALUE" x="160.02" y="96.012" size="1.778" layer="96" rot="R180"/>
-</instance>
-<instance part="R4" gate="G$1" x="152.4" y="90.17" smashed="yes" rot="R180">
-<attribute name="NAME" x="147.32" y="86.5886" size="1.778" layer="95"/>
-<attribute name="VALUE" x="160.02" y="88.392" size="1.778" layer="96" rot="R180"/>
+<instance part="R3" gate="G$1" x="152.4" y="82.55" smashed="yes" rot="R180">
+<attribute name="NAME" x="147.32" y="84.0486" size="1.778" layer="95"/>
+<attribute name="VALUE" x="160.02" y="85.852" size="1.778" layer="96" rot="R180"/>
+</instance>
+<instance part="R4" gate="G$1" x="152.4" y="80.01" smashed="yes" rot="R180">
+<attribute name="NAME" x="147.32" y="76.4286" size="1.778" layer="95"/>
+<attribute name="VALUE" x="160.02" y="78.232" size="1.778" layer="96" rot="R180"/>
 </instance>
 <instance part="R5" gate="G$1" x="167.64" y="171.45" smashed="yes" rot="R90">
@@
 <segment>
 <pinref part="R4" gate="G$1" pin="2"/>
-<wire x1="147.32" y1="90.17" x2="144.78" y2="90.17" width="0.1524" layer="91"/>
-<wire x1="144.78" y1="90.17" x2="144.78" y2="92.71" width="0.1524" layer="91"/>
+<wire x1="147.32" y1="80.01" x2="144.78" y2="80.01" width="0.1524" layer="91"/>
+<wire x1="144.78" y1="80.01" x2="144.78" y2="82.55" width="0.1524" layer="91"/>
 <pinref part="R3" gate="G$1" pin="2"/>
-<wire x1="147.32" y1="92.71" x2="144.78" y2="92.71" width="0.1524" layer="91"/>
-<wire x1="135.89" y1="92.71" x2="144.78" y2="92.71" width="0.1524" layer="91"/>
-<junction x="144.78" y="92.71"/>
-<label x="138.43" y="92.71" size="1.778" layer="95"/>
+<wire x1="147.32" y1="82.55" x2="144.78" y2="82.55" width="0.1524" layer="91"/>
+<wire x1="135.89" y1="82.55" x2="144.78" y2="82.55" width="0.1524" layer="91"/>
+<junction x="144.78" y="82.55"/>
+<label x="138.43" y="82.55" size="1.778" layer="95"/>
 </segment>
 <segment>
@@
 </segment>
 <segment>
+<pinref part="X2" gate="G$1" pin="35"/>
+<wire x1="38.1" y1="107.95" x2="25.4" y2="107.95" width="0.1524" layer="91"/>
+<label x="27.94" y="107.95" size="1.778" layer="95"/>
+</segment>
+</net>
+<net name="RXD_1" class="0">
+<segment>
+<pinref part="U1" gate="G$1" pin="RXD_1"/>
+<wire x1="175.26" y1="105.41" x2="175.26" y2="92.71" width="0.1524" layer="91"/>
+<label x="175.26" y="95.25" size="1.778" layer="95" rot="R90"/>
+</segment>
+<segment>
+<pinref part="X2" gate="G$1" pin="36"/>
+<wire x1="53.34" y1="107.95" x2="69.85" y2="107.95" width="0.1524" layer="91"/>
+<label x="58.42" y="107.95" size="1.778" layer="95"/>
+</segment>
+</net>
+<net name="RX_DV" class="0">
+<segment>
+<pinref part="R3" gate="G$1" pin="1"/>
+<pinref part="U1" gate="G$1" pin="RX_DV"/>
+<wire x1="157.48" y1="82.55" x2="162.56" y2="82.55" width="0.1524" layer="91"/>
+<wire x1="162.56" y1="82.55" x2="162.56" y2="105.41" width="0.1524" layer="91"/>
+<label x="162.56" y="91.44" size="1.778" layer="95" rot="R90"/>
+</segment>
+<segment>
 <pinref part="X2" gate="G$1" pin="33"/>
 <wire x1="38.1" y1="110.49" x2="25.4" y2="110.49" width="0.1524" layer="91"/>
@@
 </segment>
 </net>
-<net name="RXD_1" class="0">
-<segment>
-<pinref part="U1" gate="G$1" pin="RXD_1"/>
-<wire x1="175.26" y1="105.41" x2="175.26" y2="92.71" width="0.1524" layer="91"/>
-<label x="175.26" y="95.25" size="1.778" layer="95" rot="R90"/>
+<net name="CRS_DV" class="0">
+<segment>
+<pinref part="U1" gate="G$1" pin="CRS"/>
+<wire x1="165.1" y1="105.41" x2="165.1" y2="80.01" width="0.1524" layer="91"/>
+<pinref part="R4" gate="G$1" pin="1"/>
+<wire x1="157.48" y1="80.01" x2="165.1" y2="80.01" width="0.1524" layer="91"/>
+<label x="165.1" y="91.44" size="1.778" layer="95" rot="R90"/>
 </segment>
 <segment>
@@
 </segment>
 </net>
-<net name="N$1" class="0">
-<segment>
-<pinref part="R3" gate="G$1" pin="1"/>
-<pinref part="U1" gate="G$1" pin="RX_DV"/>
-<wire x1="157.48" y1="92.71" x2="162.56" y2="92.71" width="0.1524" layer="91"/>
-<wire x1="162.56" y1="92.71" x2="162.56" y2="105.41" width="0.1524" layer="91"/>
-</segment>
-</net>
-<net name="N$2" class="0">
-<segment>
-<pinref part="U1" gate="G$1" pin="CRS"/>
-<wire x1="165.1" y1="105.41" x2="165.1" y2="90.17" width="0.1524" layer="91"/>
-<pinref part="R4" gate="G$1" pin="1"/>
-<wire x1="157.48" y1="90.17" x2="165.1" y2="90.17" width="0.1524" layer="91"/>
-</segment>
-</net>

Commit message: test branch
Parts:
- added C14: 10uF, resistor:C-EUC0805
- added C15: 100nF, resistor:C-EUC0603
- added IC1: (no value), linear-technology:LT1719
- added R15: BLM, resistor:R-EU_R0603
Connections:
- new net 3V3_A: C14.1, C15.1, IC1.V+, R15.1
- new net N$1: R15.2, X3.29
- net GND: now also C14.2, C15.2, IC1.SHDN, IC1.V-
Other:
- moved on the sheet: X1
Changed lines of the file:
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@@
 <?xml version="1.0" encoding="utf-8"?>
 <!DOCTYPE eagle SYSTEM "eagle.dtd">
-<eagle version="8.0.2">
+<eagle version="7.6.0">
 <drawing>
 <settings>
@@
 <part name="GND17" library="supply1" deviceset="GND" device=""/>
 <part name="GND18" library="supply1" deviceset="GND" device=""/>
+<part name="IC1" library="linear-technology" deviceset="LT1719" device=""/>
+<part name="GND19" library="supply1" deviceset="GND" device=""/>
+<part name="R15" library="resistor" deviceset="R-EU_" device="R0603" value="BLM"/>
+<part name="C14" library="resistor" deviceset="C-EU" device="C0805" value="10uF"/>
+<part name="GND20" library="supply1" deviceset="GND" device=""/>
+<part name="C15" library="resistor" deviceset="C-EU" device="C0603" value="100nF"/>
+<part name="GND21" library="supply1" deviceset="GND" device=""/>
 </parts>
 <sheets>
@@
 </plain>
 <instances>
-<instance part="X1" gate="G$1" x="105.41" y="208.28" smashed="yes">
-<attribute name="VALUE" x="102.87" y="203.2" size="1.778" layer="96"/>
-<attribute name="NAME" x="102.87" y="211.582" size="1.778" layer="95"/>
-</instance>
-<instance part="GND1" gate="1" x="118.11" y="199.39"/>
+<instance part="X1" gate="G$1" x="82.55" y="231.14" smashed="yes">
+<attribute name="VALUE" x="80.01" y="226.06" size="1.778" layer="96"/>
+<attribute name="NAME" x="80.01" y="234.442" size="1.778" layer="95"/>
+</instance>
+<instance part="GND1" gate="1" x="95.25" y="222.25"/>
 <instance part="X6" gate="G$1" x="45.72" y="191.77" rot="R180"/>
 <instance part="X2" gate="G$1" x="45.72" y="125.73" rot="R180"/>
@@
 <instance part="GND17" gate="1" x="67.31" y="231.14" rot="R90"/>
 <instance part="GND18" gate="1" x="100.33" y="172.72"/>
+<instance part="IC1" gate="G$1" x="139.7" y="228.6"/>
+<instance part="GND19" gate="1" x="139.7" y="213.36"/>
+<instance part="R15" gate="G$1" x="22.86" y="41.91" smashed="yes">
+<attribute name="NAME" x="20.32" y="43.4086" size="1.778" layer="95"/>
+<attribute name="VALUE" x="20.32" y="38.608" size="1.778" layer="96"/>
+</instance>
+<instance part="C14" gate="G$1" x="15.24" y="36.83" smashed="yes">
+<attribute name="NAME" x="9.144" y="37.211" size="1.778" layer="95"/>
+<attribute name="VALUE" x="9.144" y="32.131" size="1.778" layer="96"/>
+</instance>
+<instance part="GND20" gate="1" x="15.24" y="26.67"/>
+<instance part="C15" gate="G$1" x="147.32" y="243.84" smashed="yes">
+<attribute name="NAME" x="148.844" y="244.221" size="1.778" layer="95"/>
+<attribute name="VALUE" x="148.844" y="239.141" size="1.778" layer="96"/>
+</instance>
+<instance part="GND21" gate="1" x="147.32" y="234.95"/>
 </instances>
 <busses>
@@
 <pinref part="X1" gate="G$1" pin="2"/>
 <pinref part="GND1" gate="1" pin="GND"/>
-<wire x1="107.95" y1="205.74" x2="118.11" y2="205.74" width="0.1524" layer="91"/>
-<wire x1="118.11" y1="205.74" x2="118.11" y2="201.93" width="0.1524" layer="91"/>
+<wire x1="85.09" y1="228.6" x2="95.25" y2="228.6" width="0.1524" layer="91"/>
+<wire x1="95.25" y1="228.6" x2="95.25" y2="224.79" width="0.1524" layer="91"/>
 </segment>
 <segment>
@@
 <wire x1="97.79" y1="177.8" x2="100.33" y2="177.8" width="0.1524" layer="91"/>
 <junction x="100.33" y="177.8"/>
+</segment>
+<segment>
+<pinref part="IC1" gate="G$1" pin="V-"/>
+<wire x1="139.7" y1="220.98" x2="139.7" y2="218.44" width="0.1524" layer="91"/>
+<pinref part="GND19" gate="1" pin="GND"/>
+<pinref part="IC1" gate="G$1" pin="SHDN"/>
+<wire x1="139.7" y1="218.44" x2="139.7" y2="215.9" width="0.1524" layer="91"/>
+<wire x1="137.16" y1="220.98" x2="137.16" y2="218.44" width="0.1524" layer="91"/>
+<wire x1="137.16" y1="218.44" x2="139.7" y2="218.44" width="0.1524" layer="91"/>
+<junction x="139.7" y="218.44"/>
+</segment>
+<segment>
+<pinref part="GND20" gate="1" pin="GND"/>
+<pinref part="C14" gate="G$1" pin="2"/>
+<wire x1="15.24" y1="29.21" x2="15.24" y2="31.75" width="0.1524" layer="91"/>
+</segment>
+<segment>
+<pinref part="C15" gate="G$1" pin="2"/>
+<pinref part="GND21" gate="1" pin="GND"/>
+<wire x1="147.32" y1="238.76" x2="147.32" y2="237.49" width="0.1524" layer="91"/>
 </segment>
 </net>
@@
 <wire x1="6.35" y1="115.57" x2="15.24" y2="115.57" width="0.1524" layer="91"/>
 <junction x="15.24" y="115.57"/>
+<label x="8.89" y="116.84" size="1.778" layer="95"/>
 </segment>
 </net>
@@
 <segment>
 <pinref part="X1" gate="G$1" pin="1"/>
-<wire x1="107.95" y1="208.28" x2="118.11" y2="208.28" width="0.1524" layer="91"/>
-<label x="109.22" y="208.28" size="1.778" layer="95"/>
+<wire x1="85.09" y1="231.14" x2="95.25" y2="231.14" width="0.1524" layer="91"/>
+<label x="86.36" y="231.14" size="1.778" layer="95"/>
 </segment>
 </net>
@@
 </segment>
 </net>
+<net name="3V3_A" class="0">
+<segment>
+<pinref part="IC1" gate="G$1" pin="V+"/>
+<wire x1="139.7" y1="236.22" x2="139.7" y2="247.65" width="0.1524" layer="91"/>
+<label x="140.97" y="251.46" size="1.778" layer="95"/>
+<pinref part="C15" gate="G$1" pin="1"/>
+<wire x1="139.7" y1="247.65" x2="139.7" y2="254" width="0.1524" layer="91"/>
+<wire x1="147.32" y1="246.38" x2="147.32" y2="247.65" width="0.1524" layer="91"/>
+<wire x1="147.32" y1="247.65" x2="139.7" y2="247.65" width="0.1524" layer="91"/>
+<junction x="139.7" y="247.65"/>
+</segment>
+<segment>
+<pinref part="C14" gate="G$1" pin="1"/>
+<wire x1="15.24" y1="39.37" x2="15.24" y2="41.91" width="0.1524" layer="91"/>
+<pinref part="R15" gate="G$1" pin="1"/>
+<wire x1="15.24" y1="41.91" x2="17.78" y2="41.91" width="0.1524" layer="91"/>
+<wire x1="6.35" y1="41.91" x2="15.24" y2="41.91" width="0.1524" layer="91"/>
+<junction x="15.24" y="41.91"/>
+<label x="8.89" y="43.18" size="1.778" layer="95"/>
+</segment>
+</net>
+<net name="N$1" class="0">
+<segment>
+<pinref part="R15" gate="G$1" pin="2"/>
+<pinref part="X3" gate="G$1" pin="29"/>
+<wire x1="27.94" y1="41.91" x2="38.1" y2="41.91" width="0.1524" layer="91"/>
+</segment>
+</net>
